Commit message: Add a basic stand for fabric mounting to the urdf

File: dingo_description/urdf/dingo-o-prefixed.urdf.xacro (robot description, xacro)
@@ -17,4 +17,5 @@
   <material name="yellow"><color rgba="0.8 0.8 0.0 1.0" /></material>
   <material name="black"><color rgba="0.15 0.15 0.15 1.0" /></material>
+  <material name="cyan"><color rgba="0 1.0 1.0 1.0"/></material>
   <xacro:macro name="wheel" params="prefix robot_prefix *joint_pose">
     <link name="${robot_prefix}${prefix}_wheel_link">
@@ -69,4 +70,42 @@
     <origin xyz="${-wheelbase/2} ${-track/2-wheel_width/2} ${wheel_vertical_offset}" rpy="0 0 0" />
   </xacro:wheel>
+  <!-- Mounting stand for fabric attachments -->
+  <xacro:macro name="fabric_stand" params="robot_prefix">
+    <link name="${robot_prefix}fabric_mount_link">
+      <visual>
+        <origin xyz="0 0 -0.358061" rpy="0 0 0"/>
+        <geometry>
+          <box size="0.05 0.05 0.716122"/>
+        </geometry>
+        <material name="cyan" />
+      </visual>
+      <collision>
+        <origin xyz="0 0 -0.358061" rpy="0 0 0"/>
+        <geometry>
+          <box size="0.05 0.05 0.716122"/>
+        </geometry>
+      </collision>
+      <inertial>
+        <origin xyz="0 0 -0.358061" rpy="0 0 0"/>
+        <mass value="2.0"/>
+        <inertia
+            ixx="0.0855449"
+            ixy="0.0"
+            ixz="0.0"
+            iyy="0.0855449"
+            iyz="0.0"
+            izz="0.083"
+        /> <!-- https://classic.gazebosim.org/tutorials?tut=build_model&cat=build_robot -->
+      </inertial>
+    </link>
+    <joint name="${robot_prefix}fabric_mount_joint" type="fixed">
+        <origin xyz="0 0 ${0.716122}" rpy="0 0 0" />  <!-- will make it 80 cm above ground. -->
+        <parent link="${robot_prefix}mid_mount"/>
+        <child link="${robot_prefix}fabric_mount_link" />
+        <!-- <axis xyz="0 0 1" /> -->
+    </joint>
+  </xacro:macro>
+  <xacro:fabric_stand robot_prefix="${robot_prefix}">
+  </xacro:fabric_stand>
   <link name="${robot_prefix}base_link"></link>
   <joint name="${robot_prefix}base_link_joint" type="fixed">
@@ -214,4 +253,10 @@
     <turnGravityOff>false</turnGravityOff>
   </gazebo>
+  <gazebo reference="${robot_prefix}fabric_mount_link">
+    <turnGravityOff>false</turnGravityOff>
+    <!-- <material>Gazebo/DarkGrey</material> -->
+    <!-- <mu1>0.0</mu1> -->
+    <!-- <mu2>0.0</mu2> -->
+  </gazebo>
   <!-- ........................................................................ -->
   <!-- ........................................................................ -->
@@ -260,7 +305,18 @@
       <frameName>map</frameName>
       <bodyName>${robot_prefix}base_link</bodyName>
+      <!-- <bodyName>${robot_prefix}fabric_mount_link</bodyName> -->  <!-- Only base link and moving links works, fixed ones don't -->
       <topicName>ground_truth/odom</topicName>
       <updateRate>50.0</updateRate>
       <gaussianNoise>0.01</gaussianNoise>
+    </plugin>
+  </gazebo>
+  <gazebo>
+    <plugin name="force_controller" filename="libgazebo_ros_force.so">
+      <alwaysOn>true</alwaysOn>
+      <updateRate>100.0</updateRate>
+      <topicName>fabric_force</topicName>
+      <bodyName>${robot_prefix}base_link</bodyName>
+      <!-- <bodyName>${robot_prefix}fabric_mount_link</bodyName> --> <!-- Only base link and moving links works, fixed ones don't -->
+      <!-- <bodyName>${robot_prefix}front_left_wheel_link</bodyName> -->
     </plugin>
   </gazebo>

Commit message: prepare simulation files for UWB sim

File: dingo_description/urdf/dingo-o-prefixed.urdf.xacro (robot description, xacro)
@@ -4,4 +4,10 @@
   <xacro:arg name="tf_prefix" default="" />
   <xacro:property name="robot_prefix" value="$(arg tf_prefix)" />
+  <!-- Args for uwb tag ids -->
+  <xacro:arg name="uwb_tag_1_id" default="0" />
+  <xacro:arg name="uwb_tag_2_id" default="1" />
+  <xacro:property name="uwb_tag_1" value="$(arg uwb_tag_1_id)" />
+  <xacro:property name="uwb_tag_2" value="$(arg uwb_tag_2_id)" />
+  <xacro:property name="uwb_tag_mass" value="0.1" />
   <xacro:property name="pacs_enabled" value="$(optenv DINGO_PACS_ENABLED 0)" />
   <xacro:property name="PI" value="3.1415926535897931" />
@@ -13,4 +19,5 @@
   <xacro:property name="wheel_width" value="0.050" />
   <xacro:property name="dummy_inertia" value="1e-09"/>
+  <material name="white"><color rgba="1.0 1.0 1.0 1.0" /></material>
   <material name="dark_grey"><color rgba="0.2 0.2 0.2 1.0" /></material>
   <material name="light_grey"><color rgba="0.4 0.4 0.4 1.0" /></material>
@@ -108,4 +115,43 @@
   <xacro:fabric_stand robot_prefix="${robot_prefix}">
   </xacro:fabric_stand>
+  <!-- UWB tag macro -->
+  <xacro:macro name="uwb_tag" params="tag_num robot_prefix *joint_pose">
+    <link name="${robot_prefix}uwb_tag_${tag_num}_link">
+      <visual>
+        <origin xyz="0 0 0" rpy="0 0 0"/>
+        <geometry>
+            <mesh filename="package://dingo_description/meshes/Decawave.stl"/>
+        </geometry>
+        <material name="white" />
+      </visual>
+      <collision>
+          <origin xyz="0 -0.013 0" rpy="0 0 0"/>
+          <geometry>
+              <box size="0.05 0.026 0.102"/>
+          </geometry>
+      </collision>
+      <inertial>
+        <origin xyz="0 0 0" rpy="0 0 0"/>
+        <mass value="${uwb_tag_mass}"/>
+        <inertia
+          ixx="1.0" ixy="0" ixz="0"
+          iyy="1.0" iyz="0"
+          izz="1.0"/>
+      </inertial>
+    </link>
+    <joint name="${robot_prefix}uwb_tag_${tag_num}_joint" type="fixed">
+      <parent link="${robot_prefix}mid_mount"/>
+      <child link="${robot_prefix}uwb_tag_${tag_num}_link" />
+      <xacro:insert_block name="joint_pose" />
+    </joint>
+  </xacro:macro>
+  <!-- Right uwb tag -->
+  <xacro:uwb_tag tag_num="1" robot_prefix="${robot_prefix}">
+    <origin xyz="0 -0.22 0.1" rpy="0 0 0"/>
+  </xacro:uwb_tag>
+  <!-- Left uwb tag -->
+  <xacro:uwb_tag tag_num="2" robot_prefix="${robot_prefix}">
+    <origin xyz="0 0.22 0.1" rpy="0 0 ${PI}"/>
+  </xacro:uwb_tag>
   <link name="${robot_prefix}base_link"></link>
   <joint name="${robot_prefix}base_link_joint" type="fixed">
@@ -253,4 +299,5 @@
     <turnGravityOff>false</turnGravityOff>
   </gazebo>
+  <!-- Fabric mount link -->
   <gazebo reference="${robot_prefix}fabric_mount_link">
     <turnGravityOff>false</turnGravityOff>
@@ -258,4 +305,26 @@
     <!-- <mu1>0.0</mu1> -->
     <!-- <mu2>0.0</mu2> -->
+  </gazebo>
+  <!-- UWB tag 1 joint -->
+  <gazebo reference="${robot_prefix}uwb_tag_1_joint">
+    <preserveFixedJoint>true</preserveFixedJoint>
+  </gazebo>
+  <!-- UWB tag 1 link -->
+  <gazebo reference="${robot_prefix}uwb_tag_1_link">
+    <turnGravityOff>false</turnGravityOff>
+    <!-- <material>Gazebo/DarkGrey</material> -->
+    <!-- <mu1>100.0</mu1> -->
+    <!-- <mu2>50.0</mu2> -->
+  </gazebo>
+  <!-- UWB tag 2 joint -->
+  <gazebo reference="${robot_prefix}uwb_tag_2_joint">
+    <preserveFixedJoint>true</preserveFixedJoint>
+  </gazebo>
+  <!-- UWB tag 2 link -->
+  <gazebo reference="${robot_prefix}uwb_tag_2_link">
+    <turnGravityOff>false</turnGravityOff>
+    <!-- <material>Gazebo/DarkGrey</material> -->
+    <!-- <mu1>100.0</mu1> -->
+    <!-- <mu2>50.0</mu2> -->
   </gazebo>
   <!-- ........................................................................ -->
@@ -280,21 +349,21 @@
   <gazebo reference="${robot_prefix}front_left_wheel_link">
     <material>Gazebo/DarkGrey</material>
-    <mu1>0.0</mu1>
-    <mu2>0.0</mu2>
+    <mu1>100.0</mu1>
+    <mu2>50.0</mu2>
   </gazebo>
   <gazebo reference="${robot_prefix}front_right_wheel_link">
     <material>Gazebo/DarkGrey</material>
-    <mu1>0.0</mu1>
-    <mu2>0.0</mu2>
+    <mu1>100.0</mu1>
+    <mu2>50.0</mu2>
   </gazebo>
   <gazebo reference="${robot_prefix}rear_left_wheel_link">
     <material>Gazebo/DarkGrey</material>
-    <mu1>0.0</mu1>
-    <mu2>0.0</mu2>
+    <mu1>100.0</mu1>
+    <mu2>50.0</mu2>
   </gazebo>
   <gazebo reference="${robot_prefix}rear_right_wheel_link">
     <material>Gazebo/DarkGrey</material>
-    <mu1>0.0</mu1>
-    <mu2>0.0</mu2>
+    <mu1>100.0</mu1>
+    <mu2>50.0</mu2>
   </gazebo>
   <!-- ........................................................................ -->
@@ -321,4 +390,36 @@
     </plugin>
   </gazebo>
+  <!-- UWB ranging simulation plugin for tag 1 -->
+  <!-- <gazebo>
+    <plugin name='libgtec_uwb_plugin' filename='libgtec_uwb_plugin.so'>
+      <tag_link>${robot_prefix}uwb_tag_1_link</tag_link>
+      <tag_id>${uwb_tag_1}</tag_id>
+      <anchor_prefix>uwb_anchor</anchor_prefix>
+      <update_rate>10</update_rate>
+      <frequency>3.9936e9</frequency>
+      <power>-14.3</power>
+      <rx_gain>2</rx_gain>
+      <noise type='gaussian'>
+          <mean>0</mean>
+          <stddev>0.0208</stddev>
+      </noise>
+    </plugin>
+  </gazebo> -->
+  <!-- UWB ranging simulation plugin for tag 2 -->
+  <!-- <gazebo>
+    <plugin name='libgtec_uwb_plugin' filename='libgtec_uwb_plugin.so'>
+      <tag_link>${robot_prefix}uwb_tag_2_link</tag_link>
+      <tag_id>${uwb_tag_2}</tag_id>
+      <anchor_prefix>uwb_anchor</anchor_prefix>
+      <update_rate>10</update_rate>
+      <frequency>3.9936e9</frequency>
+      <power>-14.3</power>
+      <rx_gain>2</rx_gain>
+      <noise type='gaussian'>
+          <mean>0</mean>
+          <stddev>0.0208</stddev>
+      </noise>
+    </plugin>
+  </gazebo> -->
   <!-- Optional standard accessories, including their simulation data. The rendering
        of these into the final description is controlled by optenv variables, which
